Commit message: fix(drones): drop misaligned propeller joints, keep body mesh only

File: drones/urdf/ardrone.urdf (robot description, URDF)
Before this commit: robot ardrone, 5 links, 4 joints
Links:
- removed link prop_0
- removed link prop_1
- removed link prop_2
- removed link prop_3
Joints:
- removed joint prop_0_joint
- removed joint prop_1_joint
- removed joint prop_2_joint
- removed joint prop_3_joint

File: drones/urdf/crazyflie2.urdf (robot description, URDF)
Before this commit: robot crazyflie2, 5 links, 4 joints
Links:
- removed link prop_0
- removed link prop_1
- removed link prop_2
- removed link prop_3
Joints:
- removed joint prop_0_joint
- removed joint prop_1_joint
- removed joint prop_2_joint
- removed joint prop_3_joint

File: drones/urdf/firefly.urdf (robot description, URDF)
Before this commit: robot firefly, 5 links, 4 joints
Links:
- removed link prop_0
- removed link prop_1
- removed link prop_2
- removed link prop_3
Joints:
- removed joint prop_0_joint
- removed joint prop_1_joint
- removed joint prop_2_joint
- removed joint prop_3_joint

File: drones/urdf/hummingbird.urdf (robot description, URDF)
Before this commit: robot hummingbird, 5 links, 4 joints
Links:
- removed link prop_0
- removed link prop_1
- removed link prop_2
- removed link prop_3
Joints:
- removed joint prop_0_joint
- removed joint prop_1_joint
- removed joint prop_2_joint
- removed joint prop_3_joint

File: drones/urdf/iris.urdf (robot description, URDF)
Before this commit: robot iris, 5 links, 4 joints
Links:
- removed link prop_0
- removed link prop_1
- removed link prop_2
- removed link prop_3
Joints:
- removed joint prop_0_joint
- removed joint prop_1_joint
- removed joint prop_2_joint
- removed joint prop_3_joint

File: drones/urdf/neo11.urdf (robot description, URDF)
Before this commit: robot neo11, 5 links, 4 joints
Links:
- removed link prop_0
- removed link prop_1
- removed link prop_2
- removed link prop_3
Joints:
- removed joint prop_0_joint
- removed joint prop_1_joint
- removed joint prop_2_joint
- removed joint prop_3_joint

File: drones/urdf/neo9.urdf (robot description, URDF)
Before this commit: robot neo9, 5 links, 4 joints
Links:
- removed link prop_0
- removed link prop_1
- removed link prop_2
- removed link prop_3
Joints:
- removed joint prop_0_joint
- removed joint prop_1_joint
- removed joint prop_2_joint
- removed joint prop_3_joint

File: drones/urdf/pelican.urdf (robot description, URDF)
Before this commit: robot pelican, 5 links, 4 joints
Links:
- removed link prop_0
- removed link prop_1
- removed link prop_2
- removed link prop_3
Joints:
- removed joint prop_0_joint
- removed joint prop_1_joint
- removed joint prop_2_joint
- removed joint prop_3_joint

Commit message: fix(drones): add proper propellers with real per-drone arm lengths

File: drones/urdf/ardrone.urdf (robot description, URDF)
Before this commit: robot ardrone, 1 links, 0 joints
Links:
- added link rotor_0_front_right; visual mesh filename=package://drones/meshes/propeller_ccw.dae scale=0.1 0.1 0.1
- added link rotor_1_back_left; visual mesh filename=package://drones/meshes/propeller_ccw.dae scale=0.1 0.1 0.1
- added link rotor_2_front_left; visual mesh filename=package://drones/meshes/propeller_cw.dae scale=0.1 0.1 0.1
- added link rotor_3_back_right; visual mesh filename=package://drones/meshes/propeller_cw.dae scale=0.1 0.1 0.1
Joints:
- added joint rotor_0_front_right_joint: type continuous, parent base_link, child rotor_0_front_right, origin xyz=0.12727922061357855 -0.12727922061357855 0.023 rpy=0 0 0, axis 0 0 1
- added joint rotor_1_back_left_joint: type continuous, parent base_link, child rotor_1_back_left, origin xyz=-0.12727922061357855 0.12727922061357855 0.023 rpy=0 0 0, axis 0 0 1
- added joint rotor_2_front_left_joint: type continuous, parent base_link, child rotor_2_front_left, origin xyz=0.12727922061357855 0.12727922061357855 0.023 rpy=0 0 0, axis 0 0 1
- added joint rotor_3_back_right_joint: type continuous, parent base_link, child rotor_3_back_right, origin xyz=-0.12727922061357855 -0.12727922061357855 0.023 rpy=0 0 0, axis 0 0 1

File: drones/urdf/crazyflie2.urdf (robot description, URDF)
Before this commit: robot crazyflie2, 1 links, 0 joints
Links:
- added link rotor_0_front_right; visual mesh filename=package://drones/meshes/propeller_ccw.dae scale=0.023 0.023 0.023
- added link rotor_1_back_left; visual mesh filename=package://drones/meshes/propeller_ccw.dae scale=0.023 0.023 0.023
- added link rotor_2_front_left; visual mesh filename=package://drones/meshes/propeller_cw.dae scale=0.023 0.023 0.023
- added link rotor_3_back_right; visual mesh filename=package://drones/meshes/propeller_cw.dae scale=0.023 0.023 0.023
Joints:
- added joint rotor_0_front_right_joint: type continuous, parent base_link, child rotor_0_front_right, origin xyz=0.0397 -0.0397 0.005 rpy=0 0 0, axis 0 0 1
- added joint rotor_1_back_left_joint: type continuous, parent base_link, child rotor_1_back_left, origin xyz=-0.0397 0.0397 0.005 rpy=0 0 0, axis 0 0 1
- added joint rotor_2_front_left_joint: type continuous, parent base_link, child rotor_2_front_left, origin xyz=0.0397 0.0397 0.005 rpy=0 0 0, axis 0 0 1
- added joint rotor_3_back_right_joint: type continuous, parent base_link, child rotor_3_back_right, origin xyz=-0.0397 -0.0397 0.005 rpy=0 0 0, axis 0 0 1

File: drones/urdf/firefly.urdf (robot description, URDF)
Before this commit: robot firefly, 1 links, 0 joints
Links:
- added link rotor_0_front_left; visual mesh filename=package://drones/meshes/propeller_ccw.dae scale=0.1 0.1 0.1
- added link rotor_1_left; visual mesh filename=package://drones/meshes/propeller_cw.dae scale=0.1 0.1 0.1
- added link rotor_2_back_left; visual mesh filename=package://drones/meshes/propeller_ccw.dae scale=0.1 0.1 0.1
- added link rotor_3_back_right; visual mesh filename=package://drones/meshes/propeller_cw.dae scale=0.1 0.1 0.1
- added link rotor_4_right; visual mesh filename=package://drones/meshes/propeller_ccw.dae scale=0.1 0.1 0.1
- added link rotor_5_front_right; visual mesh filename=package://drones/meshes/propeller_cw.dae scale=0.1 0.1 0.1
Joints:
- added joint rotor_0_front_left_joint: type continuous, parent base_link, child rotor_0_front_left, origin xyz=0.18619546181365432 0.10749999999999998 0.037 rpy=0 0 0, axis 0 0 1
- added joint rotor_1_left_joint: type continuous, parent base_link, child rotor_1_left, origin xyz=0.0 0.215 0.037 rpy=0 0 0, axis 0 0 1
- added joint rotor_2_back_left_joint: type continuous, parent base_link, child rotor_2_back_left, origin xyz=-0.18619546181365432 0.10749999999999998 0.037 rpy=0 0 0, axis 0 0 1
- added joint rotor_3_back_right_joint: type continuous, parent base_link, child rotor_3_back_right, origin xyz=-0.18619546181365432 -0.10749999999999998 0.037 rpy=0 0 0, axis 0 0 1
- added joint rotor_4_right_joint: type continuous, parent base_link, child rotor_4_right, origin xyz=0.0 -0.215 0.037 rpy=0 0 0, axis 0 0 1
- added joint rotor_5_front_right_joint: type continuous, parent base_link, child rotor_5_front_right, origin xyz=0.18619546181365432 -0.10749999999999998 0.037 rpy=0 0 0, axis 0 0 1

File: drones/urdf/hummingbird.urdf (robot description, URDF)
Before this commit: robot hummingbird, 1 links, 0 joints
Links:
- added link rotor_0_front; visual mesh filename=package://drones/meshes/propeller_cw.dae scale=0.1 0.1 0.1
- added link rotor_1_left; visual mesh filename=package://drones/meshes/propeller_ccw.dae scale=0.1 0.1 0.1
- added link rotor_2_back; visual mesh filename=package://drones/meshes/propeller_cw.dae scale=0.1 0.1 0.1
- added link rotor_3_right; visual mesh filename=package://drones/meshes/propeller_ccw.dae scale=0.1 0.1 0.1
Joints:
- added joint rotor_0_front_joint: type continuous, parent base_link, child rotor_0_front, origin xyz=0.17 0.0 0.01 rpy=0 0 0, axis 0 0 1
- added joint rotor_1_left_joint: type continuous, parent base_link, child rotor_1_left, origin xyz=0.0 0.17 0.01 rpy=0 0 0, axis 0 0 1
- added joint rotor_2_back_joint: type continuous, parent base_link, child rotor_2_back, origin xyz=-0.17 0.0 0.01 rpy=0 0 0, axis 0 0 1
- added joint rotor_3_right_joint: type continuous, parent base_link, child rotor_3_right, origin xyz=0.0 -0.17 0.01 rpy=0 0 0, axis 0 0 1

File: drones/urdf/iris.urdf (robot description, URDF)
Before this commit: robot iris, 1 links, 0 joints
Links:
- added link rotor_0_front_right; visual mesh filename=package://drones/meshes/propeller_ccw.dae scale=0.1 0.1 0.1
- added link rotor_1_back_left; visual mesh filename=package://drones/meshes/propeller_ccw.dae scale=0.1 0.1 0.1
- added link rotor_2_front_left; visual mesh filename=package://drones/meshes/propeller_cw.dae scale=0.1 0.1 0.1
- added link rotor_3_back_right; visual mesh filename=package://drones/meshes/propeller_cw.dae scale=0.1 0.1 0.1
Joints:
- added joint rotor_0_front_right_joint: type continuous, parent base_link, child rotor_0_front_right, origin xyz=0.13 -0.22 0.023 rpy=0 0 0, axis 0 0 1
- added joint rotor_1_back_left_joint: type continuous, parent base_link, child rotor_1_back_left, origin xyz=-0.13 0.2 0.023 rpy=0 0 0, axis 0 0 1
- added joint rotor_2_front_left_joint: type continuous, parent base_link, child rotor_2_front_left, origin xyz=0.13 0.22 0.023 rpy=0 0 0, axis 0 0 1
- added joint rotor_3_back_right_joint: type continuous, parent base_link, child rotor_3_back_right, origin xyz=-0.13 -0.2 0.023 rpy=0 0 0, axis 0 0 1

File: drones/urdf/neo11.urdf (robot description, URDF)
Before this commit: robot neo11, 1 links, 0 joints
Links:
- added link rotor_0_front; visual mesh filename=package://drones/meshes/neo11_propeller_cw.dae scale=0.1397 0.1397 0.1397
- added link rotor_1_left; visual mesh filename=package://drones/meshes/neo11_propeller_ccw.dae scale=0.1397 0.1397 0.1397
- added link rotor_2_back; visual mesh filename=package://drones/meshes/neo11_propeller_cw.dae scale=0.1397 0.1397 0.1397
- added link rotor_3_right; visual mesh filename=package://drones/meshes/neo11_propeller_ccw.dae scale=0.1397 0.1397 0.1397
Joints:
- added joint rotor_0_front_joint: type continuous, parent base_link, child rotor_0_front, origin xyz=0.2895 0.0 0.028 rpy=0 0 0, axis 0 0 1
- added joint rotor_1_left_joint: type continuous, parent base_link, child rotor_1_left, origin xyz=0.0 0.2895 0.028 rpy=0 0 0, axis 0 0 1
- added joint rotor_2_back_joint: type continuous, parent base_link, child rotor_2_back, origin xyz=-0.2895 0.0 0.028 rpy=0 0 0, axis 0 0 1
- added joint rotor_3_right_joint: type continuous, parent base_link, child rotor_3_right, origin xyz=0.0 -0.2895 0.028 rpy=0 0 0, axis 0 0 1

File: drones/urdf/neo9.urdf (robot description, URDF)
Before this commit: robot neo9, 1 links, 0 joints
Links:
- added link rotor_0_front; visual mesh filename=package://drones/meshes/neo9_propeller_cw.dae scale=0.1143 0.1143 0.1143
- added link rotor_1_left; visual mesh filename=package://drones/meshes/neo9_propeller_ccw.dae scale=0.1143 0.1143 0.1143
- added link rotor_2_back; visual mesh filename=package://drones/meshes/neo9_propeller_cw.dae scale=0.1143 0.1143 0.1143
- added link rotor_3_right; visual mesh filename=package://drones/meshes/neo9_propeller_ccw.dae scale=0.1143 0.1143 0.1143
Joints:
- added joint rotor_0_front_joint: type continuous, parent base_link, child rotor_0_front, origin xyz=0.2495 0.0 0.028 rpy=0 0 0, axis 0 0 1
- added joint rotor_1_left_joint: type continuous, parent base_link, child rotor_1_left, origin xyz=0.0 0.2495 0.028 rpy=0 0 0, axis 0 0 1
- added joint rotor_2_back_joint: type continuous, parent base_link, child rotor_2_back, origin xyz=-0.2495 0.0 0.028 rpy=0 0 0, axis 0 0 1
- added joint rotor_3_right_joint: type continuous, parent base_link, child rotor_3_right, origin xyz=0.0 -0.2495 0.028 rpy=0 0 0, axis 0 0 1

File: drones/urdf/pelican.urdf (robot description, URDF)
Before this commit: robot pelican, 1 links, 0 joints
Links:
- added link rotor_0_front; visual mesh filename=package://drones/meshes/propeller_cw.dae scale=0.128 0.128 0.128
- added link rotor_1_left; visual mesh filename=package://drones/meshes/propeller_ccw.dae scale=0.128 0.128 0.128
- added link rotor_2_back; visual mesh filename=package://drones/meshes/propeller_cw.dae scale=0.128 0.128 0.128
- added link rotor_3_right; visual mesh filename=package://drones/meshes/propeller_ccw.dae scale=0.128 0.128 0.128
Joints:
- added joint rotor_0_front_joint: type continuous, parent base_link, child rotor_0_front, origin xyz=0.21 0.0 0.05 rpy=0 0 0, axis 0 0 1
- added joint rotor_1_left_joint: type continuous, parent base_link, child rotor_1_left, origin xyz=0.0 0.21 0.05 rpy=0 0 0, axis 0 0 1
- added joint rotor_2_back_joint: type continuous, parent base_link, child rotor_2_back, origin xyz=-0.21 0.0 0.05 rpy=0 0 0, axis 0 0 1
- added joint rotor_3_right_joint: type continuous, parent base_link, child rotor_3_right, origin xyz=0.0 -0.21 0.05 rpy=0 0 0, axis 0 0 1
