Commit message: fix(drones): scale iris & crazyflie2 meshes (authored in mm, not m)

File: drones/urdf/crazyflie2.urdf (robot description, URDF)
Before this commit: robot crazyflie2, 5 links, 4 joints
Links:
- link base_link: geometry collision mesh filename=package://drones/meshes/crazyflie2.dae scale=0.001 0.001 0.001; visual mesh filename=package://drones/meshes/crazyflie2.dae scale=0.001 0.001 0.001

File: drones/urdf/iris.urdf (robot description, URDF)
Before this commit: robot iris, 5 links, 4 joints
Links:
- link base_link: geometry collision mesh filename=package://drones/meshes/iris.dae scale=0.001 0.001 0.001; visual mesh filename=package://drones/meshes/iris.dae scale=0.001 0.001 0.001
