Commit message: fix(drones): neo9/neo11 are hexacopters (6 rotors), not quads

File: drones/urdf/neo11.urdf (robot description, URDF)
Before this commit: robot neo11, 5 links, 4 joints
Links:
- removed link rotor_0_front
- removed link rotor_2_back
- removed link rotor_3_right
- added link rotor_0_front_left; visual mesh filename=package://drones/meshes/neo11_propeller_ccw.dae scale=0.1397 0.1397 0.1397
- added link rotor_2_back_left; visual mesh filename=package://drones/meshes/neo11_propeller_ccw.dae scale=0.1397 0.1397 0.1397
- added link rotor_3_back_right; visual mesh filename=package://drones/meshes/neo11_propeller_cw.dae scale=0.1397 0.1397 0.1397
- added link rotor_4_right; visual mesh filename=package://drones/meshes/neo11_propeller_ccw.dae scale=0.1397 0.1397 0.1397
- added link rotor_5_front_right; visual mesh filename=package://drones/meshes/neo11_propeller_cw.dae scale=0.1397 0.1397 0.1397
- link rotor_1_left: geometry visual mesh filename=package://drones/meshes/neo11_propeller_cw.dae scale=0.1397 0.1397 0.1397
Joints:
- removed joint rotor_0_front_joint
- removed joint rotor_2_back_joint
- removed joint rotor_3_right_joint
- added joint rotor_0_front_left_joint: type continuous, parent base_link, child rotor_0_front_left, origin xyz=0.247 0.1506 0.028 rpy=0.08726646259971647 0 0.5235987755982988, axis 0 0 1
- added joint rotor_2_back_left_joint: type continuous, parent base_link, child rotor_2_back_left, origin xyz=-0.247 0.1454 0.028 rpy=0.08726646259971647 0 2.6179938779914944, axis 0 0 1
- added joint rotor_3_back_right_joint: type continuous, parent base_link, child rotor_3_back_right, origin xyz=-0.247 -0.1454 0.028 rpy=-0.08726646259971647 0 -2.6179938779914944, axis 0 0 1
- added joint rotor_4_right_joint: type continuous, parent base_link, child rotor_4_right, origin xyz=-0.00067 -0.28929 0.028 rpy=0 0.08726646259971647 3.141592653589793, axis 0 0 1
- added joint rotor_5_front_right_joint: type continuous, parent base_link, child rotor_5_front_right, origin xyz=0.247 -0.1506 0.028 rpy=-0.08726646259971647 0 -0.5235987755982988, axis 0 0 1
- joint rotor_1_left_joint: origin xyz=0.0 0.2895 0.028 rpy=0 0 0 -> xyz=-0.00067 0.28929 0.028 rpy=0 -0.08726646259971647 0

File: drones/urdf/neo9.urdf (robot description, URDF)
Before this commit: robot neo9, 5 links, 4 joints
Links:
- removed link rotor_0_front
- removed link rotor_2_back
- removed link rotor_3_right
- added link rotor_0_front_left; visual mesh filename=package://drones/meshes/neo9_propeller_ccw.dae scale=0.1143 0.1143 0.1143
- added link rotor_2_back_left; visual mesh filename=package://drones/meshes/neo9_propeller_ccw.dae scale=0.1143 0.1143 0.1143
- added link rotor_3_back_right; visual mesh filename=package://drones/meshes/neo9_propeller_cw.dae scale=0.1143 0.1143 0.1143
- added link rotor_4_right; visual mesh filename=package://drones/meshes/neo9_propeller_ccw.dae scale=0.1143 0.1143 0.1143
- added link rotor_5_front_right; visual mesh filename=package://drones/meshes/neo9_propeller_cw.dae scale=0.1143 0.1143 0.1143
- link rotor_1_left: geometry visual mesh filename=package://drones/meshes/neo9_propeller_cw.dae scale=0.1143 0.1143 0.1143
Joints:
- removed joint rotor_0_front_joint
- removed joint rotor_2_back_joint
- removed joint rotor_3_right_joint
- added joint rotor_0_front_left_joint: type continuous, parent base_link, child rotor_0_front_left, origin xyz=0.213 0.12988 0.028 rpy=0.08726646259971647 0 0.5235987755982988, axis 0 0 1
- added joint rotor_2_back_left_joint: type continuous, parent base_link, child rotor_2_back_left, origin xyz=-0.21561 0.12535 0.028 rpy=0.08726646259971647 0 2.6179938779914944, axis 0 0 1
- added joint rotor_3_back_right_joint: type continuous, parent base_link, child rotor_3_back_right, origin xyz=-0.21561 -0.12535 0.028 rpy=-0.08726646259971647 0 -2.6179938779914944, axis 0 0 1
- added joint rotor_4_right_joint: type continuous, parent base_link, child rotor_4_right, origin xyz=-0.00067 -0.24939 0.028 rpy=0 0.08726646259971647 3.141592653589793, axis 0 0 1
- added joint rotor_5_front_right_joint: type continuous, parent base_link, child rotor_5_front_right, origin xyz=0.213 -0.12988 0.028 rpy=-0.08726646259971647 0 -0.5235987755982988, axis 0 0 1
- joint rotor_1_left_joint: origin xyz=0.0 0.2495 0.028 rpy=0 0 0 -> xyz=-0.00067 0.24939 0.028 rpy=0 -0.08726646259971647 0
