Commit message: fix(webots): drop double-add of HingeJoint anchor+endpoint translation

File: webots/robotti/urdf/robotti.urdf (robot description, URDF)
Before this commit: robot robotti, 42 links, 41 joints
Links:
- added link link_41; visual mesh filename=package://robotti/meshes/wheel_mount.dae
- added link link_42; visual mesh filename=package://robotti/meshes/wheel_motor.dae
- added link link_43; visual cylinder length=0.12 radius=0.071
- added link link_44; visual mesh filename=package://robotti/meshes/wheel.dae
- link link_10: geometry visual mesh filename=package://robotti/meshes/plant_camera_rack.dae
- link link_11: geometry visual mesh filename=package://robotti/meshes/plant_camera_mount.dae
- link link_12: geometry visual mesh filename=package://robotti/meshes/camera.dae
- link link_13: geometry visual mesh filename=package://robotti/meshes/plant_camera_mount.dae
- link link_14: geometry visual mesh filename=package://robotti/meshes/camera.dae
- link link_15: geometry visual mesh filename=package://robotti/meshes/plant_camera_mount.dae
- link link_16: geometry visual mesh filename=package://robotti/meshes/camera.dae
- link link_17: geometry visual mesh filename=package://robotti/meshes/plant_camera_mount.dae
- link link_18: geometry visual mesh filename=package://robotti/meshes/camera.dae
- link link_19: geometry visual mesh filename=package://robotti/meshes/camera_mount.dae
- link link_20: geometry visual mesh filename=package://robotti/meshes/camera.dae
- link link_21: geometry visual mesh filename=package://robotti/meshes/camera_mount.dae
- link link_22: geometry visual mesh filename=package://robotti/meshes/camera.dae
- link link_23: geometry visual mesh filename=package://robotti/meshes/camera_mount.dae
- link link_24: geometry visual mesh filename=package://robotti/meshes/camera.dae
- link link_25: geometry visual mesh filename=package://robotti/meshes/module.dae
- link link_26: geometry visual mesh filename=package://robotti/meshes/module_bumper.dae
- link link_27: geometry visual mesh filename=package://robotti/meshes/wheel_mount.dae
- link link_28: geometry visual mesh filename=package://robotti/meshes/wheel_motor.dae
- link link_29: geometry visual cylinder length=0.12 radius=0.071
- link link_30: geometry visual mesh filename=package://robotti/meshes/wheel.dae
- link link_31: geometry visual mesh filename=package://robotti/meshes/wheel_mount.dae
- link link_32: geometry visual mesh filename=package://robotti/meshes/wheel_motor.dae
- link link_33: geometry visual cylinder length=0.12 radius=0.071
- link link_34: geometry visual mesh filename=package://robotti/meshes/wheel.dae
- link link_35: geometry visual mesh filename=package://robotti/meshes/module.dae
- link link_36: geometry visual mesh filename=package://robotti/meshes/module_bumper.dae
- link link_37: geometry visual mesh filename=package://robotti/meshes/wheel_mount.dae
- link link_38: geometry visual mesh filename=package://robotti/meshes/wheel_motor.dae
- link link_39: geometry visual cylinder length=0.12 radius=0.071
- link link_40: geometry visual mesh filename=package://robotti/meshes/wheel.dae
- link link_6: geometry visual mesh filename=package://robotti/meshes/hitch.dae
- link link_7: geometry visual mesh filename=package://robotti/meshes/implement_mount.dae
- link link_8: geometry visual mesh filename=package://robotti/meshes/front_bumper.dae
- link link_9: geometry visual cylinder length=3.0 radius=0.009
Joints:
- added joint joint_41: type fixed, parent base_link, child link_41, origin xyz=0.0000 0.0000 0.0000 rpy=0.0000 0.0000 0.0000
- added joint joint_42: type fixed, parent base_link, child link_42, origin xyz=0.0000 0.0000 0.0000 rpy=0.0000 0.0000 0.0000
- added joint joint_43: type fixed, parent base_link, child link_43, origin xyz=0.0000 0.0000 0.0000 rpy=0.0000 0.0000 0.0000
- added joint joint_44: type fixed, parent base_link, child link_44, origin xyz=0.0000 0.0000 0.0000 rpy=0.0000 0.0000 0.0000
- joint joint_28: axis 0.0000 0.0000 1.0000 -> (none); origin xyz=0.2900 -0.1300 -0.0750 rpy=0.0000 0.0000 0.0000 -> xyz=0.0000 0.0000 0.0000 rpy=0.0000 0.0000 0.0000; type continuous -> fixed
- joint joint_29: parent link_28 -> base_link
- joint joint_30: parent link_28 -> base_link
- joint joint_31: parent link_28 -> base_link
- joint joint_32: axis 0.0000 -1.0000 0.0000 -> (none); origin xyz=0.0000 0.1300 -0.0100 rpy=0.0000 0.0000 0.0000 -> xyz=0.0000 0.0000 0.0000 rpy=0.0000 0.0000 0.0000; parent link_28 -> base_link; type continuous -> fixed
- joint joint_33: parent link_32 -> base_link
- joint joint_34: axis 0.0000 0.0000 1.0000 -> (none); origin xyz=-1.2600 -0.1300 -0.0750 rpy=0.0000 0.0000 0.0000 -> xyz=0.0000 0.0000 0.0000 rpy=0.0000 0.0000 0.0000; type continuous -> fixed
- joint joint_35: parent link_34 -> base_link
- joint joint_36: parent link_34 -> base_link
- joint joint_37: parent link_34 -> base_link
- joint joint_38: axis 0.0000 -1.0000 0.0000 -> (none); origin xyz=0.0000 0.1300 -0.0100 rpy=0.0000 0.0000 0.0000 -> xyz=0.0000 0.0000 0.0000 rpy=0.0000 0.0000 0.0000; parent link_34 -> base_link; type continuous -> fixed
- joint joint_39: parent link_38 -> base_link
- joint joint_40: axis 0.0000 1.0000 0.0000 -> (none); origin xyz=0.4850 1.5000 1.0132 rpy=0.0000 0.0000 0.0000 -> xyz=0.0000 0.0000 0.0000 rpy=0.0000 0.0000 0.0000; type continuous -> fixed
- joint joint_6: axis 0.0000 1.0000 0.0000 -> (none); origin xyz=0.1800 0.0000 -0.1600 rpy=0.0000 0.0000 0.0000 -> xyz=0.0000 0.0000 0.0000 rpy=0.0000 0.0000 0.0000; type continuous -> fixed
- joint joint_7: parent link_6 -> base_link
- joint joint_8: parent link_6 -> base_link

Commit message: fix(webots): honour Transform.scale wrappers (wheels were 1m bbox uncompensated)

File: webots/robotti/urdf/robotti.urdf (robot description, URDF)
Before this commit: robot robotti, 46 links, 45 joints
Links:
- link link_30: geometry visual mesh filename=package://robotti/meshes/wheel.dae scale=0.72 0.264 0.72
- link link_34: geometry visual mesh filename=package://robotti/meshes/wheel.dae scale=0.72 0.264 0.72
- link link_40: geometry visual mesh filename=package://robotti/meshes/wheel.dae scale=0.72 0.264 0.72
- link link_44: geometry visual mesh filename=package://robotti/meshes/wheel.dae scale=0.72 0.264 0.72
